Commit message: new launch files

File: manipulation/dual_robot_description/urdf/robot_a_.urdf.xacro (robot description, xacro)
@@ -1,10 +1,9 @@
 <?xml version="1.0"?>
 <robot xmlns:xacro="http://wiki.ros.org/xacro"
-       name="dual_viper" >
+       name="robot_a_" >
   <!-- Robot -->
   <xacro:include filename="$(find dual_robot_description)/urdf/robot.urdf.xacro" />
   <!-- arm -->
   <xacro:vx300s prefix="robot_a_"/>
-  <xacro:vx300s prefix="robot_b_"/>
   <link name="world"/>
     <joint name="robot_a_to_world" type="fixed">
@@ -12,9 +11,4 @@
       <child link="robot_a_base_link"/>
       <origin xyz="0 0.15 0" />
-    </joint>
-    <joint name="robot_b_to_world" type="fixed">
-      <parent link="world"/>
-      <child link="robot_b_base_link"/>
-      <origin xyz="0 -0.15 0" />
     </joint>
   <gazebo>
@@ -25,10 +19,3 @@
     </plugin>
   </gazebo>
-  <gazebo>
-    <plugin name="gazebo_ros_control" filename="libgazebo_ros_control.so">
-      <robotSimType>gazebo_ros_control/DefaultRobotHWSim</robotSimType>
-      <legacyModeNS>true</legacyModeNS>
-      <robotNamespace>/robot_b_</robotNamespace>
-    </plugin>
-  </gazebo>
 </robot>

File: manipulation/dual_robot_description/urdf/robot_b_.urdf.xacro (robot description, xacro)
@@ -1,16 +1,10 @@
 <?xml version="1.0"?>
 <robot xmlns:xacro="http://wiki.ros.org/xacro"
-       name="dual_viper" >
+       name="robot_b_" >
   <!-- Robot -->
   <xacro:include filename="$(find dual_robot_description)/urdf/robot.urdf.xacro" />
   <!-- arm -->
-  <xacro:vx300s prefix="robot_a_"/>
   <xacro:vx300s prefix="robot_b_"/>
   <link name="world"/>
-    <joint name="robot_a_to_world" type="fixed">
-      <parent link="world"/>
-      <child link="robot_a_base_link"/>
-      <origin xyz="0 0.15 0" />
-    </joint>
     <joint name="robot_b_to_world" type="fixed">
       <parent link="world"/>
@@ -22,11 +16,4 @@
       <robotSimType>gazebo_ros_control/DefaultRobotHWSim</robotSimType>
       <legacyModeNS>true</legacyModeNS>
-      <robotNamespace>/robot_a_</robotNamespace>
-    </plugin>
-  </gazebo>
-  <gazebo>
-    <plugin name="gazebo_ros_control" filename="libgazebo_ros_control.so">
-      <robotSimType>gazebo_ros_control/DefaultRobotHWSim</robotSimType>
-      <legacyModeNS>true</legacyModeNS>
       <robotNamespace>/robot_b_</robotNamespace>
     </plugin>
