Commit message: working dual arm control on real robots

File: manipulation/dual_robot_description/urdf/dual_robot.urdf.xacro (robot description, xacro)
@@ -11,16 +11,16 @@
       <parent link="world"/>
       <child link="robot_a_base_link"/>
-      <origin xyz="0 0.15 0" />
+      <origin xyz="0 -0.15 0" />
     </joint>
     <joint name="robot_b_to_world" type="fixed">
       <parent link="world"/>
       <child link="robot_b_base_link"/>
-      <origin xyz="0 -0.15 0" />
+      <origin xyz="0 0.15 0" />
     </joint>
-  <gazebo>
+  <!--<gazebo>
     <plugin name="gazebo_ros_control" filename="libgazebo_ros_control.so">
       <robotSimType>gazebo_ros_control/DefaultRobotHWSim</robotSimType>
       <legacyModeNS>true</legacyModeNS>
     </plugin>
-  </gazebo>
+  </gazebo>-->
 </robot>

File: manipulation/dual_robot_description/urdf/robot.urdf.xacro (robot description, xacro)
@@ -2,6 +2,4 @@
 <robot  xmlns:xacro="http://ros.org/wiki/xacro">
 <xacro:macro name="vx300s" params="prefix ">
-  <xacro:arg name="robot_name" default = "vx300s"/>
-  <xacro:arg name="base_link_frame" default="base_link"/>
   <xacro:arg name="show_gripper_bar" default="true"/>
   <xacro:arg name="show_gripper_fingers" default="true"/>

File: manipulation/dual_robot_description/urdf/robot_a_.urdf.xacro (robot description, xacro)
@@ -12,5 +12,5 @@
       <origin xyz="0 0.15 0" />
     </joint>
-  <gazebo>
+  <!--<gazebo>
     <plugin name="gazebo_ros_control" filename="libgazebo_ros_control.so">
       <robotSimType>gazebo_ros_control/DefaultRobotHWSim</robotSimType>
@@ -18,4 +18,4 @@
       <robotNamespace>/robot_a_</robotNamespace>
     </plugin>
-  </gazebo>
+  </gazebo>-->
 </robot>

Commit message: first stable version of wire grasping framework

File: manipulation/dual_robot_description/urdf/dual_robot.urdf.xacro (robot description, xacro)
@@ -11,10 +11,10 @@
       <parent link="world"/>
       <child link="robot_a_base_link"/>
-      <origin xyz="0 -0.15 0" />
+      <origin xyz="0 -0.1778 0" />
     </joint>
     <joint name="robot_b_to_world" type="fixed">
       <parent link="world"/>
       <child link="robot_b_base_link"/>
-      <origin xyz="0 0.15 0" />
+      <origin xyz="0 0.1778 0" />
     </joint>
   <gazebo>
@@ -24,3 +24,57 @@
     </plugin>
   </gazebo>
+  <link name="panel_1">
+    <inertial>
+    <origin xyz="0 0 0" rpy="0 0 0"/>
+    <mass value="1"/>
+      <inertia ixx="100"  ixy="0"  ixz="0" iyy="100" iyz="0" izz="100" />
+      </inertial>
+      <visual>
+        <origin xyz="0 0 0" rpy="0 0 0" />
+        <geometry>
+          <box size="0.02 0.762 0.6096" />
+        </geometry>
+          <material name="Cyan">
+        <color rgba="0 1.0 1.0 1.0"/>
+          </material>
+      </visual>
+      <collision>
+        <origin xyz="0 0 0" rpy="0 0 0"/>
+          <geometry>
+            <box size="0.02 0.762 0.6096" />
+          </geometry>
+      </collision>
+    </link>
+    <link name="panel_2">
+    <inertial>
+    <origin xyz="0 0 0" rpy="0 0 0"/>
+    <mass value="1"/>
+      <inertia ixx="100"  ixy="0"  ixz="0" iyy="100" iyz="0" izz="100" />
+      </inertial>
+      <visual>
+        <origin xyz="0 0 0" rpy="0 0 0" />
+        <geometry>
+          <box size="0.4572 0.02 0.6096" />
+        </geometry>
+          <material name="Cyan">
+        <color rgba="0 1.0 1.0 1.0"/>
+          </material>
+      </visual>
+      <collision>
+        <origin xyz="0 0 0" rpy="0 0 0"/>
+          <geometry>
+            <box size="0.4572 0.02 0.6096" />
+          </geometry>
+      </collision>
+    </link>
+    <joint name="panel_joint" type="fixed">
+      <parent link="panel_1"/>
+      <child link="panel_2"/>
+      <origin xyz="-0.2286 -0.391 0" />
+    </joint>
+    <joint name="panel_to_world" type="fixed">
+      <parent link="world"/>
+      <child link="panel_1"/>
+      <origin xyz="0.4921 -0.0381 0.3048" />
+    </joint>
 </robot>

Commit message: improvments to vision and simulator. Added experimental testing

File: manipulation/dual_robot_description/urdf/dual_robot.urdf.xacro (robot description, xacro)
@@ -76,5 +76,5 @@
       <parent link="world"/>
       <child link="panel_1"/>
-      <origin xyz="0.4921 -0.0381 0.3048" />
+      <origin xyz="0.5334 -0.0381 0.3048" />
     </joint>
 </robot>
