Commit message: Fixes + adding 2nd realsense

File: wire_manipulation_description/urdf/base_scene.xacro (robot description, xacro)
@@ -8,4 +8,10 @@
   <!-- VX300s macro -->
   <xacro:include filename="$(find vx300s_description)/urdf/vx300s_macro.xacro" />
+  <!-- realsense macro -->
+  <xacro:include filename="$(find realsense2_description)/urdf/_d415.urdf.xacro" />
+  <!-- realsense d415 -->
+  <xacro:sensor_d415 name="b_bot" parent="b_bot_ee_arm_link" use_nominal_extrinsics="true">
+    <origin xyz="-0.05 0 0.05" />
+  </xacro:sensor_d415>
   <!-- dual vx300s, a_bot and b_bot -->
   <xacro:vx300s prefix="a_bot_" hw_interface="hardware_interface/EffortJointInterface" />

Commit message: Arm cam frame adjustments

File: wire_manipulation_description/urdf/base_scene.xacro (robot description, xacro)
@@ -11,7 +11,8 @@
   <xacro:include filename="$(find realsense2_description)/urdf/_d415.urdf.xacro" />
   <!-- realsense d415 -->
-  <xacro:sensor_d415 name="b_bot" parent="b_bot_ee_arm_link" use_nominal_extrinsics="true">
-    <origin xyz="-0.05 0 0.05" />
+  <xacro:sensor_d415 name="b_bot" parent="b_bot_gripper_link" use_nominal_extrinsics="true">
+    <origin xyz="-0.0254 0 0.0635" />
   </xacro:sensor_d415>
+  <!-- b_bot_link, b_bot_gripper_link 3" -->
   <!-- dual vx300s, a_bot and b_bot -->
   <xacro:vx300s prefix="a_bot_" hw_interface="hardware_interface/EffortJointInterface" />

Commit message: Frame error fix and adjusting mounted cam position

File: wire_manipulation_description/urdf/base_scene.xacro (robot description, xacro)
@@ -9,9 +9,14 @@
   <xacro:include filename="$(find vx300s_description)/urdf/vx300s_macro.xacro" />
   <!-- realsense macro -->
-  <xacro:include filename="$(find realsense2_description)/urdf/_d415.urdf.xacro" />
+  <xacro:include filename="$(find wire_manipulation_description)/urdf/realsense/d415.urdf.xacro" />
+  <xacro:include filename="$(find realsense2_description)/urdf/_d435i.urdf.xacro" />
   <!-- realsense d415 -->
   <xacro:sensor_d415 name="d415" parent="b_bot_gripper_link" use_nominal_extrinsics="true">
     <origin xyz="-0.0254 0 0.0635" />
   </xacro:sensor_d415>
+  <xacro:sensor_d435i name="d435i" parent="world" use_nominal_extrinsics="true">
+    <origin xyz="${-0.3556 - 0.0106} ${0.0 - 0.0325} ${0.4064 - 0.0125}" />
+  </xacro:sensor_d435i>
+  <!-- 0.0106; 0.0325; 0.0125 -->
   <!-- dual vx300s, a_bot and b_bot -->
   <xacro:vx300s prefix="a_bot_" hw_interface="hardware_interface/EffortJointInterface" />

Commit message: Arm cam frame adjustments

File: wire_manipulation_description/urdf/base_scene.xacro (robot description, xacro)
@@ -12,7 +12,9 @@
   <xacro:include filename="$(find realsense2_description)/urdf/_d435i.urdf.xacro" />
   <!-- realsense d415 -->
-  <xacro:sensor_d415 name="d415" parent="b_bot_gripper_link" use_nominal_extrinsics="true">
-    <origin xyz="-0.0254 0 0.0635" />
+  <xacro:sensor_d415 name="d415" parent="b_bot_wrist_link" use_nominal_extrinsics="true">
+    <origin xyz="0.0762 0 0.0635" />
+    <!-- <origin xyz="-1 0 1" /> -->
   </xacro:sensor_d415>
+  <!-- want position offset from b_bot_gripper_link and rotation of b_bot_wrist_link -->
   <xacro:sensor_d435i name="d435i" parent="world" use_nominal_extrinsics="true">
     <origin xyz="${-0.3556 - 0.0106} ${0.0 - 0.0325} ${0.4064 - 0.0125}" />

Commit message: Adjust new cam position on b_bot_ee_arm_link

File: wire_manipulation_description/urdf/base_scene.xacro (robot description, xacro)
@@ -12,6 +12,6 @@
   <xacro:include filename="$(find realsense2_description)/urdf/_d435i.urdf.xacro" />
   <!-- realsense d415 -->
-  <xacro:sensor_d415 name="d415" parent="b_bot_wrist_link" use_nominal_extrinsics="true">
-    <origin xyz="0.0762 0 0.0635" />
+  <xacro:sensor_d415 name="d415" parent="b_bot_ee_arm_link" use_nominal_extrinsics="true">
+    <origin xyz="0.0127 0 0.0635" />
     <!-- <origin xyz="-1 0 1" /> -->
   </xacro:sensor_d415>

Commit message: Swap cameras with functional segmenting

File: wire_manipulation_description/urdf/base_scene.xacro (robot description, xacro)
@@ -11,13 +11,12 @@
   <xacro:include filename="$(find wire_manipulation_description)/urdf/realsense/d415.urdf.xacro" />
   <xacro:include filename="$(find realsense2_description)/urdf/_d435i.urdf.xacro" />
-  <!-- realsense d415 -->
-  <xacro:sensor_d415 name="d415" parent="b_bot_ee_arm_link" use_nominal_extrinsics="true">
+  <!-- realsense d435i -->
+  <xacro:sensor_d435i name="d435i" parent="b_bot_ee_arm_link" use_nominal_extrinsics="true">
     <origin xyz="0.0127 0 0.0635" />
     <!-- <origin xyz="-1 0 1" /> -->
+  </xacro:sensor_d435i>
+  <xacro:sensor_d415 name="d415" parent="world" use_nominal_extrinsics="true">
+    <origin xyz="${-0.3556 - 0.0106} ${0.0 - 0.0325} ${0.4064 - 0.0125}" />
   </xacro:sensor_d415>
-  <!-- want position offset from b_bot_gripper_link and rotation of b_bot_wrist_link -->
-  <xacro:sensor_d435i name="d435i" parent="world" use_nominal_extrinsics="true">
-    <origin xyz="${-0.3556 - 0.0106} ${0.0 - 0.0325} ${0.4064 - 0.0125}" />
-  </xacro:sensor_d435i>
   <!-- 0.0106; 0.0325; 0.0125 -->
   <!-- dual vx300s, a_bot and b_bot -->
